File: mixed_signal_hardware_design.kicad_sch (KiCad schematic)
At the start: 0 parts

Commit message: Added sub schematic, was not added in previous commit
Other:
- added sheet ADC (adc.kicad_sch)
- added sheet DAC (dac.kicad_sch)
- added sheet MCU (mcu.kicad_sch)
- added sheet Power (power.kicad_sch)
- note added: "Mixed-Signal PCB Learning Project"
- note added: "[1] Power"
- note added: "[2] MCU"
- note added: "[3] ADC"
- note added: "[4] DAC"
Changed lines of the file:
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@@
 		(rev "0.1")
+	)
+	(text "[2] MCU"
+		(exclude_from_sim no)
+		(at 179.578 41.402 0)
+		(effects
+			(font
+				(size 5 5)
+				(thickness 1)
+				(bold yes)
+			)
+		)
+	)
+	(text "Mixed-Signal PCB Learning Project"
+		(exclude_from_sim no)
+		(at 91.948 22.86 0)
+		(effects
+			(font
+				(size 5 5)
+				(thickness 1)
+				(bold yes)
+			)
+		)
+	)
+	(text "[4] DAC\n"
+		(exclude_from_sim no)
+		(at 179.07 105.41 0)
+		(effects
+			(font
+				(size 5 5)
+				(thickness 1)
+				(bold yes)
+			)
+		)
+	)
+	(text "[3] ADC"
+		(exclude_from_sim no)
+		(at 90.17 105.156 0)
+		(effects
+			(font
+				(size 5 5)
+				(thickness 1)
+				(bold yes)
+			)
+		)
+	)
+	(text "[1] Power"
+		(exclude_from_sim no)
+		(at 93.98 41.91 0)
+		(effects
+			(font
+				(size 5 5)
+				(thickness 1)
+				(bold yes)
+			)
+		)
+	)
+	(sheet
+		(at 165.1 50.8)
+		(size 38.1 39.37)
+		(fields_autoplaced yes)
+		(stroke
+			(width 0.1524)
+			(type solid)
+		)
+		(fill
+			(color 0 0 0 0.0000)
+		)
+		(property "Sheetname" "MCU"
+			(at 165.1 50.0884 0)
+			(effects
+				(font
+					(size 1.27 1.27)
+				)
+				(justify left bottom)
+			)
+		)
+		(property "Sheetfile" "mcu.kicad_sch"
+			(at 165.1 90.7546 0)
+			(effects
+				(font
+					(size 1.27 1.27)
+				)
+				(justify left top)
+			)
+		)
+		(instances
+			(project "mixed_signal_hardware_design"
+				(path "/eba96202-8ea2-41d9-8d7a-700a4166585a"
+					(page "3")
+				)
+			)
+		)
+	)
+	(sheet
+		(at 165.1 114.3)
+		(size 38.1 38.1)
+		(fields_autoplaced yes)
+		(stroke
+			(width 0.1524)
+			(type solid)
+		)
+		(fill
+			(color 0 0 0 0.0000)
+		)
+		(property "Sheetname" "DAC"
+			(at 165.1 113.5884 0)
+			(effects
+				(font
+					(size 1.27 1.27)
+				)
+				(justify left bottom)
+			)
+		)
+		(property "Sheetfile" "dac.kicad_sch"
+			(at 165.1 152.9846 0)
+			(effects
+				(font
+					(size 1.27 1.27)
+				)
+				(justify left top)
+			)
+		)
+		(instances
+			(project "mixed_signal_hardware_design"
+				(path "/eba96202-8ea2-41d9-8d7a-700a4166585a"
+					(page "5")
+				)
+			)
+		)
+	)
+	(sheet
+		(at 76.2 50.8)
+		(size 38.1 38.1)
+		(fields_autoplaced yes)
+		(stroke
+			(width 0.1524)
+			(type solid)
+		)
+		(fill
+			(color 0 0 0 0.0000)
+		)
+		(property "Sheetname" "Power"
+			(at 76.2 50.0884 0)
+			(effects
+				(font
+					(size 1.27 1.27)
+				)
+				(justify left bottom)
+			)
+		)
+		(property "Sheetfile" "power.kicad_sch"
+			(at 76.2 89.4846 0)
+			(effects
+				(font
+					(size 1.27 1.27)
+				)
+				(justify left top)
+			)
+		)
+		(instances
+			(project "mixed_signal_hardware_design"
+				(path "/eba96202-8ea2-41d9-8d7a-700a4166585a"
+					(page "2")
+				)
+			)
+		)
+	)
+	(sheet
+		(at 76.2 114.3)
+		(size 38.1 38.1)
+		(fields_autoplaced yes)
+		(stroke
+			(width 0.1524)
+			(type solid)
+		)
+		(fill
+			(color 0 0 0 0.0000)
+		)
+		(property "Sheetname" "ADC"
+			(at 76.2 113.5884 0)
+			(effects
+				(font
+					(size 1.27 1.27)
+				)
+				(justify left bottom)
+			)
+		)
+		(property "Sheetfile" "adc.kicad_sch"
+			(at 76.2 152.9846 0)
+			(effects
+				(font
+					(size 1.27 1.27)
+				)
+				(justify left top)
+			)
+		)
+		(instances
+			(project "mixed_signal_hardware_design"
+				(path "/eba96202-8ea2-41d9-8d7a-700a4166585a"
+					(page "4")
+				)
+			)
+		)
 	)
 	(sheet_instances
