File: kicad/mcu.kicad_sch (KiCad schematic)
At the start: 0 parts

Commit message: Added schematic for MCU
Parts:
- added C10: 10u, symbol Device:C
- added C11, C12, C13, C14, C20, C21, C22: 100n, symbol Device:C
- added C15: 10n, symbol Device:C
- added C16, C17: 1u, symbol Device:C
- added C18, C19: 10p, symbol Device:C
- added D2: LED_RGBA, symbol Device:LED_RGBA
- added D3, D4, D5, D6, D7: ~, symbol CMF3216F-900-2P-T:D_TVS
- added J1: USB_C_Receptacle_USB2.0_16P, symbol Connector:USB_C_Receptacle_USB2.0_16P
- added J2: 2x5x1.27mm, symbol Connector_Generic:Conn_02x05_Counter_Clockwise
- added L3: 10n, symbol Device:L
- added L4: CMF3216F-900-2P-T, Inductor_SMD:L_CommonMode_Wurth_WE-CNSW-1206, symbol Filter:Choke_Wurth_WE-CNSW_744232090
- added R10, R7, R9: 10k, symbol Device:R
- added R11: 0R, symbol Device:R
- added R12, R13, R14: 1k, symbol Device:R
- added R15, R16: 5k1, symbol Device:R
- added R17, R18, R19, R20: 49R9, symbol Device:R
- added R8: 1k5, symbol Device:R
- added U4: STM32F103CBT6, Package_QFP:LQFP-48_7x7mm_P0.5mm, symbol MCU_ST_STM32F1:STM32F103CBTx
- added U5: USBLC6-2SC6, Package_TO_SOT_SMD:SOT-23-6, symbol Power_Protection:USBLC6-2SC6
- added Y1: 16MHz, symbol Device:Crystal_GND24
Connections:
- new net: D4.2 (A2), J2.10 (Pin_10), R17.1
- new net: D5.2 (A2), J2.9 (Pin_9), R18.1
- new net: D6.2 (A2), J2.8 (Pin_8), R19.1
- new net: D7.2 (A2), J2.6 (Pin_6), R20.1
- new net +3V3: C10.1, C11.1, C12.1, C13.1, C14.1, C17.1, C20.1, D2.2 (A), D3.2 (A2), J2.1 (Pin_1), L3.2, R10.1, R7.1, R8.1, U4.1 (VBAT), U4.24 (VDD), U4.36 (VDD), U4.48 (VDD)
- new net BOOT0: R9.2, U4.44 (BOOT0)
- new net DAC_NCLR: U4.21 (PB10)
- new net DAC_NLDAC: U4.22 (PB11)
- new net GND: C10.2, C11.2, C12.2, C13.2, C14.2, C15.2, C16.2, C17.2, C18.2, C19.2, C20.2, C21.1, C22.2, D3.1 (A1), D4.1 (A1), D5.1 (A1), D6.1 (A1), D7.1 (A1), J1.A1 (GND), J1.A12 (GND), J1.B1 (GND), J1.B12 (GND), J2.2 (Pin_2), J2.3 (Pin_3), J2.5 (Pin_5), R15.2, R16.2, R9.1, U4.23 (VSS), U4.35 (VSS), U4.47 (VSS), U4.8 (VSSA), U5.2 (GND), Y1.2, Y1.4
- new net HSE_IN: C19.1, U4.5 (PD0), Y1.1
- new net HSE_OUT: R11.2, U4.6 (PD1)
- new net LED_B_K: D2.4 (BK), R14.2
- new net LED_G_K: D2.1 (GK), R13.2
- new net LED_R_K: D2.3 (RK), R12.2
- new net NRST: C22.1, R20.2, U4.7 (NRST)
- new net SPI1_MISO: U4.16 (PA6)
- new net SPI1_NSS: R7.2, U4.14 (PA4)
- new net SPI1_SCK: U4.15 (PA5)
- new net SPI2_MISO: U4.28 (PB15)
- new net SPI2_NSS: R10.2, U4.25 (PB12)
- new net SPI2_SCK: U4.26 (PB13)
- new net SWCLK: R18.2, U4.37 (PA14)
- new net SWDIO: R17.2, U4.34 (PA13)
- new net SWO: R19.2, U4.39 (PB3)
- new net TIM4_CH1: R12.1, U4.42 (PB6)
- new net TIM4_CH2: R13.1, U4.43 (PB7)
- new net TIM4_CH3: R14.1, U4.45 (PB8)
- new net UBS_CONN_D-: J1.A7 (D-), J1.B7 (D-)
- new net USB_CMC_D+: L4.2, U5.4 (I/O2)
- new net USB_CMC_D-: L4.1, U5.6 (I/O1)
- new net USB_CONN_CC1: J1.A5 (CC1), R15.1
- new net USB_CONN_CC2: J1.B5 (CC2), R16.1
- new net USB_CONN_D+: J1.A6 (D+), J1.B6 (D+), U5.3 (I/O2)
- new net USB_CONN_D-: U5.1 (I/O1)
- new net USB_D+: L4.3, R8.2, U4.33 (PA12)
- new net USB_D-: L4.4, U4.32 (PA11)
- new net VBUS: C21.2, J1.A4 (VBUS), J1.A9 (VBUS), J1.B4 (VBUS), J1.B9 (VBUS), U5.5 (VBUS)
- new net VDDA: C15.1, C16.1, L3.1, U4.9 (VDDA)
- new net XTAL_IN: C18.1, R11.1, Y1.3
- no-connect marks 0 -> 24
Other:
- note added: "CL=10pF ESR=80R"
- note added: "Common-Mode Choke Impedence: 90R"
- note added: "Crystal App Note: AN2867"
- note added: "MCU (STM32F1)"
- note added: "PESD3V3L1BA,115"
- note added: "RGB LED"
- note added: "SWD Connector"
- note added: "Signal Path: Connector <-> ESD Protection <-> Common-Mode Choke <-> Pull-Up <-> MCU"
- note added: "USB App Note: AN4879"
- note added: "USB Type C"
- note added: "[2] Microcontroller & USB"
